File: EspNow Vibration Sensor/hardware/vibration_sensor/vibration_sensor.kicad_sch (KiCad schematic)
At the start: 29 parts, among them U1 TLV9062

Commit message: ongoing changes to vibration sensor
Parts:
- C10, C11, C4: value 10u -> 1u; footprint (none) -> Capacitor_THT:CP_Radial_D5.0mm_P2.50mm
- C12, C5: footprint (none) -> Capacitor_THT:CP_Radial_D5.0mm_P2.50mm
- C13, C3, C7, C8, C9, Cc1: footprint (none) -> Capacitor_THT:C_Disc_D8.0mm_W5.0mm_P7.50mm
- C2: value 1u -> 0.1u; footprint (none) -> Capacitor_THT:C_Disc_D8.0mm_W5.0mm_P7.50mm
- R1, R10, R11, R2, R3, R4, R5, R6, R7, R8, R9a1, R9b1: footprint (none) -> Resistor_THT:R_Axial_DIN0309_L9.0mm_D3.2mm_P12.70mm_Horizontal
Connections:
- net PIEZO_A: now reaches C2.1, Piezo1.1 (Pin1)
Other:
- note added: "ATtiny13A Always-On Wake Trigger (raw piezo tap, powers analog + ESP rails)"

Commit message: complete sensor in working condition. Schematic is also final.
Parts:
- added C6: 10u, Capacitor_THT:CP_Radial_D5.0mm_P2.50mm, symbol Device:C_Polarized
- added HT1: HT7333, Package_TO_SOT_THT:TO-92, symbol custom_symbol_library:HT7333
- added J1: Serial(G,Rx,Tx), Connector_JST:JST_XH_B2B-XH-A_1x02_P2.50mm_Vertical, symbol Connector_Generic:Conn_01x03
- added J1: Batt, Connector_JST:JST_XH_B2B-XH-A_1x02_P2.50mm_Vertical, symbol Connector:Conn_01x02_Pin
- added R12, R9: 3K3, Resistor_THT:R_Axial_DIN0309_L9.0mm_D3.2mm_P12.70mm_Horizontal, symbol Device:R
- added U2: ESP-12E, RF_Module:ESP-12E, symbol RF_Module:ESP-12E
- Piezo1: footprint (none) -> Connector_Molex:Molex_KK-254_AE-6410-02A_1x02_P2.54mm_Vertical
- U1: footprint (none) -> custom_footprint_library:tl9062_dip
Connections:
- net GND: now also C6.2, HT1.1 (Gnd), J1.1 (Pin_1), J1.1 (Pin_1), U2.15 (GND), U2.16 (GPIO15)
- net +3.3V: no longer names the net of C8.2, D1.1 (K), R1.1, R7.1, U1.8 (V+)
- net +3.3V: now also U2.19 (GPIO4)
- net To Bare ESP ADC (0-1V): no longer names the net of C4.1, R9a1.2, R9b1.1
- net To Bare ESP ADC (0-1V): now also U2.2 (ADC)
- net VBIAS: no longer names the net of C10.1, C3.1, C7.1, C9.2, R1.2, R2.1, R3.2
- net VLOW: no longer names the net of C11.1, C13.2, R10.1, R7.2, R8.1
- new net: HT1.2 (Vin), J1.2 (Pin_2)
- new net: C6.1, HT1.3 (Vout), R12.1, R9.1, U2.8 (VCC)
- new net: R9.2, U2.1 (~{RST}), U2.4 (GPIO16)
- new net: J1.2 (Pin_2), U2.21 (GPIO3/RXD)
- new net: J1.3 (Pin_3), U2.22 (GPIO1/TXD)
- new net: R12.2, U2.3 (EN)
Other:
- note removed: "ATtiny13A Always-On Wake Trigger (raw piezo tap, powers analog + ESP rails)"
